File: hardware/Handheld-Gaming-Device.kicad_pcb (KiCad board)
At the start: 2 copper layers, 256.5 x 139.5 mm, 25 parts, among them J1 SNAP Programmer, J2 Right Joystick, J3 Left Joystick, J4 OLED, J5 USB input, J6 Voltage Regulator, Q1 2N2219, SW1 Red Button, SW2 Blue Button, U1 PIC24FJ64GA002-I/SP

Commit message: PCB design change
Changed the layout and size of the PCB
Parts:
- moved RV1 58.8 mm to (188.0, 65.0)
- moved R3 56.5 mm to (196.5, 68.2)
- moved R2 56.0 mm to (196.5, 54.2)
- moved LS1 56.0 mm to (196.5, 36.0)
- moved J3 55.5 mm to (201.8, 96.5)
- moved R4 55.5 mm to (186.5, 44.9)
- moved Q1 54.5 mm to (183.9, 36.5)
- moved C5 44.1 mm to (187.0, 73.0), turned to 180 degrees
- moved J2 35.4 mm to (113.3, 96.0)
- moved SW2 33.8 mm to (191.0, 99.5)
- moved C4 32.6 mm to (199.5, 73.0), turned to 180 degrees
- moved SW1 23.5 mm to (176.5, 99.5)
- moved C8 19.5 mm to (82.0, 38.5), turned to 90 degrees
- moved C7 15.1 mm to (79.0, 32.5)
- moved R5 13.4 mm to (199.9, 83.0)
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Routing:
- net +3V3: track 739.2 -> 514.3 mm
- net Net-(J3-Pin_3): track 274.9 -> 187.0 mm
- net Net-(J3-Pin_4): track 273.6 -> 188.6 mm
- net Net-(J2-Pin_3): track 145.5 -> 96.7 mm
- net Net-(J2-Pin_2): track 150.4 -> 102.5 mm
- net Net-(J2-Pin_4): track 131.0 -> 84.8 mm
- net Net-(C4-Pad2): track 9.21 -> 34.8 mm
- net Net-(R5-Pad1): track 132.0 -> 118.6 mm
- net +5V: track 32.4 -> 19.3 mm
- net Net-(Q1-B): track 16.1 -> 5.90 mm
- net Net-(C5-Pad2): track 3.98 -> 13.7 mm
- net GND: track 20.2 -> 11.8 mm
- net Net-(R4-Pad2): track 15.4 -> 7.99 mm
- net Net-(SW2-Pad2): track 96.0 -> 88.8 mm
- net Net-(R2-Pad1): track 9.34 -> 3.84 mm
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Other:
- board size 256.5 x 139.5 mm -> 153.7 x 94.2 mm
